File: templates/kicad/T24-10/T24-10.kicad_pcb (KiCad board)
At the start: 2 copper layers, 2 x 4 mm, 10 parts

Commit message: Re-tier on measured prices: 4L on 0.2 mm drill, add 4L-fine
4L keeps the 0.2 mm drill so it lands in PCBWay's $162 standard bucket
rather than the $419 one; 3/3 mil and 0.15 mm drills move to a new 4L-fine
tier on the advanced form. Quotes name the calculator to use. set_tier.py
gains --package for projects that predate the templates and --ignore-locks
for stale lock files.

Co-Authored-By: Claude Fable 5.1 <noreply@anthropic.com>
Other:
- board text added: "T24-10 2-layer standard ORDER AT PCBWAY AS: Standard calculator: 2 layers / 0.4 mm / 4/4 mil / min hole 0.2 mm / ENIG / tenting FR-4 0.4 mm, 1 oz Cu, ENIG, green mask, white silk (bottom only) track/space >= 0.1 mm, copper to edge >= 0.15 mm (base pads excepted) via 0.4/0.2 mm, hole-to-hole >= 0.25, copper-to-hole >= 0.15 components top side only; bottom = base pads + name pinout: P1=GND, P4=I2C.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"
- board text removed: "T24-10 2-layer standard ORDER AT PCBWAY AS: 2 layers / 0.4 mm / 4/4 mil / min hole 0.2 mm / ENIG FR-4 0.4 mm, 1 oz Cu, ENIG, green mask, white silk (bottom only) track/space >= 0.1 mm, copper to edge >= 0.15 mm (base pads excepted) via 0.4/0.2 mm, hole-to-hole >= 0.25, copper-to-hole >= 0.15 components top side only; bottom = base pads + name pinout: P1=GND, P4=I2C.CLK, P5=I2C.DAT, P10=+V"
Changed lines of the file:
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@@
 		(layer "User.4")
 	)
-	(gr_text "T24-10  2-layer standard\nORDER AT PCBWAY AS: 2 layers / 0.4 mm / 4/4 mil / min hole 0.2 mm / ENIG\nFR-4 0.4 mm, 1 oz Cu, ENIG, green mask, white silk (bottom only)\ntrack/space >= 0.1 mm, copper to edge >= 0.15 mm (base pads excepted)\nvia 0.4/0.2 mm, hole-to-hole >= 0.25, copper-to-hole >= 0.15\ncomponents top side only; bottom = base pads + name\npinout: P1=GND, P4=I2C.CLK, P5=I2C.DAT, P10=+V"
+	(gr_text "T24-10  2-layer standard\nORDER AT PCBWAY AS: Standard calculator: 2 layers / 0.4 mm / 4/4 mil / min hole 0.2 mm / ENIG / tenting\nFR-4 0.4 mm, 1 oz Cu, ENIG, green mask, white silk (bottom only)\ntrack/space >= 0.1 mm, copper to edge >= 0.15 mm (base pads excepted)\nvia 0.4/0.2 mm, hole-to-hole >= 0.25, copper-to-hole >= 0.15\ncomponents top side only; bottom = base pads + name\npinout: P1=GND, P4=I2C.CLK, P5=I2C.DAT, P10=+V"
 		(at 3 -2 0)
 		(layer "Cmts.User")

Commit message: Solder mask dam 0.19 mm, from PCBWay DFM feedback
Co-Authored-By: Claude Fable 5.1 <noreply@anthropic.com>
Other:
- rule solder_mask_min_width: 0.1 -> 0.19
Changed lines of the file:
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@@
 		)
 		(pad_to_mask_clearance 0)
-		(solder_mask_min_width 0.1)
+		(solder_mask_min_width 0.19)
 		(allow_soldermask_bridges_in_footprints no)
 		(tenting front back)
